File: giggle.kicad_pcb (KiCad board)
At the start: 2 copper layers, 100 x 100 mm, 41 parts

Commit message: finished the side, i guess.
Parts:
- removed >NAME: >VALUE, connector-shrouded
- added J2: CONN_05X2SHD, connector-shrouded, F.Cu at (113.5, 38.5)
- moved sw0:0 25.7 mm to (38.1, 57.1)
- moved sw0:1 25.7 mm to (38.1, 76.2)
- moved sw0:2 25.7 mm to (38.1, 95.2)
- moved sw0:3 25.7 mm to (38.1, 114.2)
- moved sw1:0 25.7 mm to (57.1, 57.1)
- moved sw1:1 25.7 mm to (57.1, 76.2)
- moved sw1:2 25.7 mm to (57.1, 95.2)
- moved sw1:3 25.7 mm to (57.1, 114.2)
- moved sw2:1 25.7 mm to (76.1, 76.2)
- moved sw2:2 25.7 mm to (76.1, 95.2)
- moved sw2:3 25.7 mm to (76.1, 114.2)
- moved sw3:1 25.7 mm to (95.1, 76.2)
- moved sw3:2 25.7 mm to (95.1, 95.2)
- moved sw3:3 25.7 mm to (95.1, 114.2)
- moved sw4:1 25.7 mm to (114.1, 76.2)
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Connections:
- sw0:0 pad 1: N-col-0 -> N-diode-0
- sw0:0 pad 2: N-diode-0 -> N-col-0
- sw0:1 pad 1: N-col-0 -> N-diode-1
- sw0:1 pad 2: N-diode-1 -> N-col-0
- sw0:2 pad 1: N-col-0 -> N-diode-2
- sw0:2 pad 2: N-diode-2 -> N-col-0
- sw0:3 pad 1: N-col-0 -> N-diode-3
- sw0:3 pad 2: N-diode-3 -> N-col-0
- sw1:0 pad 1: N-col-1 -> N-diode-4
- sw1:0 pad 2: N-diode-4 -> N-col-1
- sw1:1 pad 1: N-col-1 -> N-diode-5
- sw1:1 pad 2: N-diode-5 -> N-col-1
- sw1:2 pad 1: N-col-1 -> N-diode-6
- sw1:2 pad 2: N-diode-6 -> N-col-1
- sw1:3 pad 1: N-col-1 -> N-diode-7
- sw1:3 pad 2: N-diode-7 -> N-col-1
- sw2:0 pad 1: N-col-2 -> N-diode-8
- sw2:0 pad 2: N-diode-8 -> N-col-2
- sw2:1 pad 1: N-col-2 -> N-diode-9
- sw2:1 pad 2: N-diode-9 -> N-col-2
- sw2:2 pad 1: N-col-2 -> N-diode-10
- sw2:2 pad 2: N-diode-10 -> N-col-2
- sw2:3 pad 1: N-col-2 -> N-diode-11
- sw2:3 pad 2: N-diode-11 -> N-col-2
- sw3:0 pad 1: N-col-3 -> N-diode-12
- sw3:0 pad 2: N-diode-12 -> N-col-3
- sw3:1 pad 1: N-col-3 -> N-diode-13
- sw3:1 pad 2: N-diode-13 -> N-col-3
- sw3:2 pad 1: N-col-3 -> N-diode-14
- sw3:2 pad 2: N-diode-14 -> N-col-3
- sw3:3 pad 1: N-col-3 -> N-diode-15
- sw3:3 pad 2: N-diode-15 -> N-col-3
- sw4:0 pad 1: N-col-4 -> N-diode-16
- sw4:0 pad 2: N-diode-16 -> N-col-4
- sw4:1 pad 1: N-col-4 -> N-diode-17
- sw4:1 pad 2: N-diode-17 -> N-col-4
- sw4:2 pad 1: N-col-4 -> N-diode-18
- sw4:2 pad 2: N-diode-18 -> N-col-4
- sw4:3 pad 1: N-col-4 -> N-diode-19
- sw4:3 pad 2: N-diode-19 -> N-col-4
Routing:
- net N-row-3: track 0.00 -> 182.1 mm
- net N-row-2: track 0.00 -> 159.4 mm
- net N-col-0: track 0.00 -> 140.7 mm
- net N-row-1: track 0.00 -> 136.0 mm
- net N-col-1: track 0.00 -> 127.3 mm
- net N-row-0: track 0.45 -> 112.8 mm
- net N-col-2: track 0.00 -> 110.8 mm
- net N-col-4: track 0.00 -> 102.9 mm
- net N-col-3: track 0.00 -> 94.3 mm
- net N-diode-3: track 0.00 -> 7.65 mm
- net N-diode-2: track 0.00 -> 7.65 mm
- net N-diode-1: track 0.00 -> 7.65 mm
- net N-diode-0: track 0.00 -> 7.65 mm
- net N-diode-6: track 0.00 -> 7.65 mm
- net N-diode-19: track 0.00 -> 7.65 mm
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Other:
- board size 100 x 100 mm -> 97.5 x 97 mm
